File: DS100M08KV2.kicad_pcb (KiCad board)
At the start: 2 copper layers, 100 x 52 mm, 180 parts, among them J1 wire2board, J10 BNC_panel_mount, J11 wire2board, J2 Conn_01x04_Socket, J3 wire2board, J4 wire2board, J5 USB_C_floating, J8 red_safety_4mm_connector, J9 black_safety_4mm_connector, Q1 MMBT5401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

Commit message: Some errors fixed.
Parts:
- added C68: 20p, Resistor_SMD:R_0603_1608Metric_Pad0.98x0.95mm_HandSolder, F.Cu at (125.2, 160.2)
- added C69: 10p, Resistor_SMD:R_0603_1608Metric_Pad0.98x0.95mm_HandSolder, F.Cu at (125.2, 162.7)
- added C70: 10p, Resistor_SMD:R_0603_1608Metric_Pad0.98x0.95mm_HandSolder, F.Cu at (125.2, 165.2)
- added C71: 33p, Resistor_SMD:R_0603_1608Metric_Pad0.98x0.95mm_HandSolder, F.Cu at (125.2, 167.7)
- added C72: 20p, Resistor_SMD:R_0603_1608Metric_Pad0.98x0.95mm_HandSolder, F.Cu at (125.2, 170.2)
- added C73: 10p, Resistor_SMD:R_0603_1608Metric_Pad0.98x0.95mm_HandSolder, F.Cu at (125.2, 172.8)
- added C74: 10p, Resistor_SMD:R_0603_1608Metric_Pad0.98x0.95mm_HandSolder, F.Cu at (137.6, 131.6)
- added C75: 10p, Resistor_SMD:R_0603_1608Metric_Pad0.98x0.95mm_HandSolder, F.Cu at (137.6, 134.1)
- added C76: 10p, Resistor_SMD:R_0603_1608Metric_Pad0.98x0.95mm_HandSolder, F.Cu at (153.6, 166.9)
- added C77: 12p, Resistor_SMD:R_0603_1608Metric_Pad0.98x0.95mm_HandSolder, F.Cu at (153.6, 169.4)
- added C78: 15p, Resistor_SMD:R_0603_1608Metric_Pad0.98x0.95mm_HandSolder, F.Cu at (153.6, 171.9)
- added C79: 18p, Resistor_SMD:R_0603_1608Metric_Pad0.98x0.95mm_HandSolder, F.Cu at (153.6, 174.4)
- added C80: 20p, Resistor_SMD:R_0603_1608Metric_Pad0.98x0.95mm_HandSolder, F.Cu at (157.9, 161.9)
- added C81: 22p, Resistor_SMD:R_0603_1608Metric_Pad0.98x0.95mm_HandSolder, F.Cu at (157.9, 164.4)
- added C82: 30p, Resistor_SMD:R_0603_1608Metric_Pad0.98x0.95mm_HandSolder, F.Cu at (157.9, 166.9)
- added C83: 47p, Resistor_SMD:R_0603_1608Metric_Pad0.98x0.95mm_HandSolder, F.Cu at (157.9, 169.4)
- added C84: 10p, Resistor_SMD:R_0603_1608Metric_Pad0.98x0.95mm_HandSolder, F.Cu at (157.9, 171.9)
- added C85: 12p, Resistor_SMD:R_0603_1608Metric_Pad0.98x0.95mm_HandSolder, F.Cu at (157.9, 174.4)
- added C86: 15p, Resistor_SMD:R_0603_1608Metric_Pad0.98x0.95mm_HandSolder, F.Cu at (162.2, 161.9)
- added C87: 18p, Resistor_SMD:R_0603_1608Metric_Pad0.98x0.95mm_HandSolder, F.Cu at (162.2, 164.4)
- added C88: 20p, Resistor_SMD:R_0603_1608Metric_Pad0.98x0.95mm_HandSolder, F.Cu at (162.2, 166.9)
- added C89: 22p, Resistor_SMD:R_0603_1608Metric_Pad0.98x0.95mm_HandSolder, F.Cu at (162.2, 169.4)
- added C90: 30p, Resistor_SMD:R_0603_1608Metric_Pad0.98x0.95mm_HandSolder, F.Cu at (162.2, 171.9)
- added C91: 47p, Resistor_SMD:R_0603_1608Metric_Pad0.98x0.95mm_HandSolder, F.Cu at (162.2, 174.4)
- C25, C56: value 100p -> 47p
- C58: value 10p -> 33p
- R36: value 10k -> 2.2k
- turned R36 to 180 degrees
Connections:
- D13 pad 1: -BATT -> Earth
- R36 pad 1: Net-(U6-ISET) -> Earth
- R36 pad 2: Earth -> Net-(U6-ISET)
- U6 pad 2: -BATT -> +BATT
Routing:
- net -BATT: track 97.9 -> 73.9 mm, vias 4 -> 3
- net +BATT: track 87.9 -> 93.0 mm
