File: DS100M08KV2.kicad_sch (KiCad schematic)
At the start: 85 parts, among them J1 wire2board, J10 BNC_panel_mount, J11 wire2board, J3 wire2board, J4 wire2board, J8 red_safety_4mm_connector, J9 black_safety_4mm_connector, SW1 SW_DPDT_x2, U1 RS8752XK

Commit message: Some errors fixed.
Parts:
- added C68, C72, C80, C88: 20p, Resistor_SMD:R_0603_1608Metric_Pad0.98x0.95mm_HandSolder, symbol Device:C
- added C69, C70, C73, C74, C75, C76, C84: 10p, Resistor_SMD:R_0603_1608Metric_Pad0.98x0.95mm_HandSolder, symbol Device:C
- added C71: 33p, Resistor_SMD:R_0603_1608Metric_Pad0.98x0.95mm_HandSolder, symbol Device:C
- added C77, C85: 12p, Resistor_SMD:R_0603_1608Metric_Pad0.98x0.95mm_HandSolder, symbol Device:C
- added C78, C86: 15p, Resistor_SMD:R_0603_1608Metric_Pad0.98x0.95mm_HandSolder, symbol Device:C
- added C79, C87: 18p, Resistor_SMD:R_0603_1608Metric_Pad0.98x0.95mm_HandSolder, symbol Device:C
- added C81, C89: 22p, Resistor_SMD:R_0603_1608Metric_Pad0.98x0.95mm_HandSolder, symbol Device:C
- added C82, C90: 30p, Resistor_SMD:R_0603_1608Metric_Pad0.98x0.95mm_HandSolder, symbol Device:C
- added C83, C91: 47p, Resistor_SMD:R_0603_1608Metric_Pad0.98x0.95mm_HandSolder, symbol Device:C
- C25, C56: value 100p -> 47p; LCSC C14858 -> C1648
- C58: value 10p -> 33p; LCSC C1634 -> C1663
Connections:
- net at C11.1, C25.2, C57.2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: now also C68.2, C69.2, C71.2
- net at C26.2, C37.2, C38.2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: now also C72.2, C73.2, C74.2
- net at C15.1, C56.1, C58.1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: now also C72.1, C73.1, C75.1
- net at C21.1, C22.1, C23.2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: now also C68.1, C70.1, C71.1
- new net: C74.1, C75.2
- new net: C69.1, C70.2
- no-connect marks 0 -> 32
Other:
- moved on the sheet: C32, C57, C66, C67, C7, C8, D1, D3, D4, D5, H4, R14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
