File: DS20M05V.kicad_pcb (KiCad board)
At the start: 2 copper layers, 100 x 52 mm, 204 parts, among them J1 wire2board, J10 BNC_panel_mount, J11 wire2board, J2 Conn_01x04_Socket, J3 wire2board, J4 wire2board, J5 USB_C_floating, J8 red_safety_4mm_connector, J9 black_safety_4mm_connector, Q1 MMBT5401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

Commit message: s
Parts:
- removed R41, R43, R44, R47: 470k, Resistor_SMD:R_0603_1608Metric_Pad0.98x0.95mm_HandSolder
- removed R45, R46, R48, R49: 1Meg, Resistor_SMD:R_0603_1608Metric_Pad0.98x0.95mm_HandSolder
- added TP10: TestPoint, TestPoint:TestPoint_Pad_D2.0mm, F.Cu at (197.3, 128.1)
- added TP11: TestPoint, TestPoint:TestPoint_Pad_D2.0mm, F.Cu at (197.3, 132.2)
- added TP12: TestPoint, TestPoint:TestPoint_Pad_D2.0mm, F.Cu at (197.3, 136.2)
- J2: footprint Connector_JST:JST_PH_B4B-PH-K_1x04_P2.00mm_Vertical -> Connector_JST:JST_EH_B4B-EH-A_1x04_P2.50mm_Vertical
- moved BT1 5.00 mm to (155.0, 126.0)
- moved RV2 2.00 mm to (123.6, 128.6)
Routing:
- net +BATT: track 93.0 -> 88.7 mm
- net -BATT: track 73.9 -> 70.2 mm
- net Net-(R12-Pad1): track 4.02 -> 2.03 mm
- net Net-(R5-Pad1): track 4.13 -> 2.27 mm
- net Earth: track 41.2 -> 42.0 mm, vias 14 -> 15

Commit message: right angle 4 mm
Parts:
- removed J4: wire2board, Connector_Wire:SolderWire-0.25sqmm_1x01_D0.65mm_OD1.7mm
- removed R12, R5: 10k, Resistor_SMD:R_0603_1608Metric_Pad0.98x0.95mm_HandSolder
- removed R31, R54: 100, Resistor_SMD:R_0603_1608Metric_Pad0.98x0.95mm_HandSolder
- added D14: PSM712-LF-T7, Package_TO_SOT_SMD:SOT-23_Handsoldering, F.Cu at (90.1, 161.0)
- added J6: Banana connector, DS20M05V:CT3151SP2-BLACK, B.Cu at (119.0, 133.0)
- added R41: 100k, Resistor_SMD:R_0603_1608Metric_Pad0.98x0.95mm_HandSolder, F.Cu at (99.7, 164.6)
- added R43: 200k, Resistor_SMD:R_0603_1608Metric_Pad0.98x0.95mm_HandSolder, F.Cu at (99.7, 167.1)
- J3: value wire2board -> Banana connector; footprint Connector_Wire:SolderWire-0.25sqmm_1x01_D0.65mm_OD1.7mm -> DS20M05V:CT3151SP2-RED; moved to B.Cu
- R13: value 82k -> 200k
- R16: value 10k -> 100k
- R18: value 82k -> 1Meg
- R6: value 10k -> 1Meg
- RV2: value 100 -> 5k
- moved J8 87.2 mm to (55.7, 68.2)
- moved J9 87.2 mm to (55.7, 44.2)
- moved H4 35.0 mm to (194.9, 108.5)
- moved J3 18.1 mm to (119.0, 119.0)
- moved BT1 12.3 mm to (167.3, 125.4)
- moved C11 7.00 mm to (128.8, 112.8)
- moved C15 7.00 mm to (128.8, 139.4)
- moved D6 7.00 mm to (134.8, 149.0)
- moved R11 7.00 mm to (128.8, 136.7)
- moved R3 7.00 mm to (128.8, 115.3)
- moved C1 7.00 mm to (186.4, 140.8)
- moved C10 7.00 mm to (123.6, 112.8)
- moved C12 7.00 mm to (113.2, 139.4)
- moved C13 7.00 mm to (118.4, 139.4)
- moved C14 7.00 mm to (123.6, 139.4)
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Connections:
- C11 pad 1: Net-(C11-Pad1) -> Net-(SW1A-B)
- C25 pad 1: Net-(C21-Pad1) -> unconnected-(C25-Pad1)
- C25 pad 2: Net-(C11-Pad1) -> unconnected-(C25-Pad2)
- C57 pad 1: Net-(C21-Pad1) -> unconnected-(C57-Pad1)
- C57 pad 2: Net-(C11-Pad1) -> unconnected-(C57-Pad2)
- C68 pad 1: Net-(C21-Pad1) -> unconnected-(C68-Pad1)
- C68 pad 2: Net-(C11-Pad1) -> unconnected-(C68-Pad2)
- C69 pad 2: Net-(C11-Pad1) -> unconnected-(C69-Pad2)
- C70 pad 1: Net-(C21-Pad1) -> unconnected-(C70-Pad1)
- C71 pad 1: Net-(C21-Pad1) -> unconnected-(C71-Pad1)
- C71 pad 2: Net-(C11-Pad1) -> unconnected-(C71-Pad2)
- R13 pad 1: Net-(C21-Pad1) -> unconnected-(R13-Pad1)
- R16 pad 1: Net-(R16-Pad1) -> Net-(C26-Pad2)
- R16 pad 2: Net-(C26-Pad2) -> Net-(C15-Pad1)
- R18 pad 1: Net-(C15-Pad1) -> Net-(R18-Pad1)
- R18 pad 2: Net-(R16-Pad1) -> Net-(C26-Pad2)
- R3 pad 2: Net-(C11-Pad1) -> Net-(SW1A-B)
- R6 pad 2: Net-(C11-Pad1) -> unconnected-(R6-Pad2)
- R7 pad 1: Net-(C11-Pad1) -> Net-(SW1A-B)
- RV2 pad 1: Net-(R12-Pad1) -> Net-(C26-Pad2)
- RV2 pad 3: Net-(R5-Pad1) -> Net-(C21-Pad1)
- SW1 pad 1: Net-(SW1A-A) -> unconnected-(SW1A-A-Pad1)
- TP1 pad 1: Net-(C11-Pad1) -> Net-(SW1A-B)
Routing:
- net Net-(C11-Pad1): track 16.6 -> 0.00 mm
- net (no net): track 0.00 -> 16.6 mm
- net unconnected-(SW1A-A-Pad1): track 0.00 -> 7.72 mm
- net Net-(SW1A-A): track 7.72 -> 0.00 mm
- net Net-(C26-Pad2): track 15.4 -> 18.9 mm
- net Net-(C39-Pad1): track 3.47 -> 0.00 mm
- net Net-(C10-Pad2): track 3.38 -> 6.85 mm
- net Net-(C21-Pad1): track 15.2 -> 17.5 mm
- net Net-(R5-Pad1): track 2.27 -> 0.00 mm
- net Net-(R12-Pad1): track 2.03 -> 0.00 mm
- net Net-(R16-Pad1): track 1.47 -> 0.00 mm
Other:
- outline, holes or cut-outs redrawn
