File: DS20M05V.kicad_sch (KiCad schematic)
At the start: 109 parts, among them J1 wire2board, J10 BNC_panel_mount, J11 wire2board, J3 wire2board, J4 wire2board, J8 red_safety_4mm_connector, J9 black_safety_4mm_connector, SW1 SW_DPDT_x2, U1 RS8752XK

Commit message: s
Parts:
- added R41: 100k, Resistor_SMD:R_0603_1608Metric_Pad0.98x0.95mm_HandSolder, symbol Device:R
- added R43: 200k, Resistor_SMD:R_0603_1608Metric_Pad0.98x0.95mm_HandSolder, symbol Device:R
- R13: value 82k -> 200k; LCSC (none) -> C25811
- R16: value 10k -> 100k; LCSC (none) -> C25803
- R18: value 82k -> 1Meg; LCSC (none) -> C22935
- R6: value 10k -> 1Meg; LCSC (none) -> C22935
Connections:
- net at C21.1, C22.1, C23.2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: now also R41.2
- net at C11.1, C25.2, C57.2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: now also R41.1
- net at C26.2, C37.2, C38.2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: now also R16.1, R18.2; no longer R16.2
- net at C15.1, C56.1, C58.1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: now also R16.2, R43.1; no longer R18.1
- new net: R18.1, R43.2
Other:
- moved on the sheet: R13, R6

Commit message: right angle 4 mm
Parts:
- removed J4: wire2board, Connector_Wire:SolderWire-0.25sqmm_1x01_D0.65mm_OD1.7mm, symbol Connector:Conn_01x01_Pin
- removed R12, R5: 10k, Resistor_SMD:R_0603_1608Metric_Pad0.98x0.95mm_HandSolder, symbol Device:R
- removed R31, R54: 100, Resistor_SMD:R_0603_1608Metric_Pad0.98x0.95mm_HandSolder, symbol Device:R
- added J6: Banana connector, DS20M05V:CT3151SP2-BLACK, symbol Connector:Conn_01x01_Pin
- J3: value wire2board -> Banana connector; footprint Connector_Wire:SolderWire-0.25sqmm_1x01_D0.65mm_OD1.7mm -> DS20M05V:CT3151SP2-RED
- RV2: value 100 -> 5k
Connections:
- net IN-: now also J6.1 (Pin_1)
- net at C21.1, C22.1, C23.2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: now also RV2.3; no longer C25.1, C57.1, C68.1, C70.1, C71.1, R13.1
- net at C26.2, C37.2, C38.2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: now also RV2.1
- net at D7.3 (K), SW1.2 (B), U1.5 (+): now also C11.1, R3.2, R7.1, TP1.1
- net at SW1.3 (C): now also R41.1
- now unconnected: C25.2, C57.2, C68.2, C69.2, C71.2, R6.2
Other:
- moved on the sheet: C25, C57, C68, C69, C70, C71, D7, J1, J10, J11, J3, R13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
