File: power_supply.kicad_sch (KiCad schematic)
At the start: 95 parts, among them J2 Conn_01x04_Socket, J5 USB_C_floating, Q1 MMBT5401, Q10 AO3401A, Q13 AO3400A, Q14 AO3400A, Q2 MMBT5551L, Q3 AO3400A, Q4 MMBT5401, Q5 AO3400A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

Commit message: Some errors fixed.
Parts:
- added TP10, TP11, TP12: TestPoint, TestPoint:TestPoint_Pad_D2.0mm, symbol Connector:TestPoint
- R36: value 10k -> 2.2k; LCSC C25804 -> C4190
Connections:
- net +BATT: now also U6.2 (OUT), TP12.1
- net -BATT: now also TP11.1; no longer D13.1 (K), U6.2 (OUT)
- net Earth: now also D13.1 (K), R36.1, TP10.1; no longer R36.2
- net at U6.4 (ISET): now also R36.2; no longer R36.1

Commit message: s
Parts:
- removed R41, R43, R44, R47: 470k, Resistor_SMD:R_0603_1608Metric_Pad0.98x0.95mm_HandSolder, symbol Device:R
- removed R45, R46, R48, R49: 1Meg, Resistor_SMD:R_0603_1608Metric_Pad0.98x0.95mm_HandSolder, symbol Device:R
- added D14: PSM712-LF-T7, Package_TO_SOT_SMD:SOT-23_Handsoldering, symbol Device:D_Zener_Dual_CommonAnode_KKA
- J2: footprint Connector_JST:JST_PH_B4B-PH-K_1x04_P2.00mm_Vertical -> Connector_JST:JST_EH_B4B-EH-A_1x04_P2.50mm_Vertical
Other:
- moved on the sheet: BT1, SW2A, SW2B, TP10, TP11, TP12

Commit message: merge
Parts:
- removed C16, C20, C36, C44, C61, C62, C63, C64: 47u, Capacitor_THT:CP_Radial_D5.0mm_P2.00mm, symbol Device:C_Polarized_US
- removed J2: Conn_01x04_Socket, Connector_JST:JST_EH_B4B-EH-A_1x04_P2.50mm_Vertical, symbol Connector:Conn_01x04_Socket
- removed J5: USB_C_floating, DS100M08KV:USB_C_floating, symbol DS100M08KV:USB_C_floating
- added BT2: Battery_Cell, DS100M08KV:battery_holder, symbol Device:Battery_Cell
- added C16, C20, C36, C44, C61, C62, C63, C64, C92, C93, C94, C95, C96: 10u, Resistor_SMD:R_0805_2012Metric_Pad1.20x1.40mm_HandSolder, symbol Device:C
- added D15: GREEN_LED, LED_SMD:LED_0805_2012Metric_Pad1.15x1.40mm_HandSolder, symbol Device:LED
- added J3: USB_C_Receptacle_PowerOnly_6P, Connector_USB:USB_C_Receptacle_GCT_USB4125-xx-x-0190_6P_TopMnt_Horizontal, symbol Connector:USB_C_Receptacle_PowerOnly_6P
- D6: value LED -> GREEN_LED; footprint LED_THT:LED_D3.0mm_FlatTop -> LED_SMD:LED_0805_2012Metric_Pad1.15x1.40mm_HandSolder; LCSC (none) -> C2297
Connections:
- net +2.5V: now also C93.2
- net +BATT: now also BT2.1 (+)
- net +VBUS: now also J3.A9 (VBUS), J3.B9 (VBUS)
- net +VIN: now also D6.2 (A), C63.2, C64.2, C94.2, C95.2, C96.2
- net -2.5V: now also C36.1
- net -BATT: now also BT2.2 (-)
- net -VIN: now also C61.2, C62.2
- net 0: now also C16.1, C20.2, C36.2, C44.2, C92.1, C93.1
- net Earth: now also C61.1, C62.1, C63.1, C64.1, C94.1, C95.1, C96.1, J3.A12 (GND), J3.B12 (GND), J3.S1 (SHIELD)
- net at Q2.1 (B), Q6.3 (C), R33.1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: now also C16.2, C92.2
- net at Q1.1 (B), Q4.3 (C), R28.1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: now also C20.1, C44.1
- net at R26.1: now also D15.2 (A); no longer D6.2 (A)
- net at U6.3 (~{CHG}): now also D15.1 (K); no longer D6.1 (K)
- no-connect marks 2 -> 0
Other:
- moved on the sheet: BT1, C2, C28, C40, Q3, Q5, R25, R26, R29, R30, R36, U2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
